File: DMH_Slew_Mk2_PANEL/DMH_Slew_Mk2_PANEL.kicad_pcb (KiCad board)
At the start: 2 copper layers, 50 x 200 mm, 28 parts

Commit message: Redesigned panel and main PCB schematic
Parts:
- removed H23: R/RF/F, SynthStuff:Toggle_Switch_TE_Cutout
- H17: value Rise A -> Slew A; footprint SynthStuff:Pot_Cutout_Small -> SynthStuff:Pot_Cutout_Medium
- H18: value Fall A -> Mod; footprint SynthStuff:Pot_Cutout_Small -> SynthStuff:Jack_6.35mm_Cutout_v3
- moved H18 93.1 mm to (91.5, 175.8)
- moved H24 36.9 mm to (91.5, 159.2)
- moved H27 29.1 mm to (79.0, 86.0)
- moved H21 26.2 mm to (91.5, 83.2)
- moved H13 16.5 mm to (58.5, 159.2)
- moved H14 16.5 mm to (75.0, 159.2)
- moved H15 16.5 mm to (58.5, 175.8)
- moved H16 16.5 mm to (75.0, 175.8)
- moved H17 9.85 mm to (75.0, 61.0)
- moved H29 3.61 mm to (71.0, 86.0)
- moved H26 0.25 mm to (58.5, 83.2)
