File: DMH_Slew_Mk2_PANEL/DMH_Slew_Mk2_PANEL.kicad_sch (KiCad schematic)
At the start: 31 parts, among them J0 Panel_GND_Solder_Wire_Pad

Commit message: Redesigned panel and main PCB schematic
Parts:
- removed H18: Fall A, SynthStuff:Pot_Cutout_Small, symbol SynthStuff:MountingHole_Pot
- removed H23: R/RF/F, SynthStuff:Toggle_Switch_TE_Cutout, symbol SynthStuff:MountingHole_ToggleSwitch
- added H18: Mod, SynthStuff:Jack_6.35mm_Cutout_v3, symbol SynthStuff:MountingHole_Jack6.35mm_v2
- H17: value Rise A -> Slew A; footprint SynthStuff:Pot_Cutout_Small -> SynthStuff:Pot_Cutout_Medium
Connections:
- net GND: now also H18.1
Changed lines of the file:
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@@
-	)
-	(junction
-		(at 63.5 120.65)
-		(diameter 0)
-		(color 0 0 0 0)
 	)
 	(junction
@@
 	)
 	(junction
-		(at 38.1 160.02)
-		(diameter 0)
-		(color 0 0 0 0)
-	)
-	(junction
 		(at 31.75 171.45)
 		(diameter 0)
@@
 	)
 	(junction
+		(at 31.75 152.4)
+		(diameter 0)
+		(color 0 0 0 0)
+	)
+	(junction
 		(at 63.5 139.7)
 		(diameter 0)
@@
 	(wire
 		(pts
-			(xy 63.5 120.65) (xy 88.9 120.65)
+			(xy 38.1 120.65) (xy 88.9 120.65)
 		)
 		(stroke
@@
 	(wire
 		(pts
-			(xy 31.75 139.7) (xy 31.75 160.02)
-		)
-		(stroke
-			(width 0)
-			(type default)
-		)
-	)
-	(wire
-		(pts
-			(xy 38.1 160.02) (xy 31.75 160.02)
+			(xy 31.75 139.7) (xy 31.75 152.4)
 		)
 		(stroke
@@
 	(wire
 		(pts
-			(xy 63.5 118.11) (xy 63.5 120.65)
+			(xy 31.75 152.4) (xy 34.29 152.4)
 		)
 		(stroke
@@
 	(wire
 		(pts
-			(xy 63.5 120.65) (xy 38.1 120.65)
-		)
-		(stroke
-			(width 0)
-			(type default)
-		)
-	)
-	(wire
-		(pts
 			(xy 31.75 120.65) (xy 31.75 139.7)
 		)
@@
 	(wire
 		(pts
+			(xy 31.75 152.4) (xy 31.75 160.02)
+		)
+		(stroke
+			(width 0)
+			(type default)
+		)
+	)
+	(wire
+		(pts
 			(xy 63.5 139.7) (xy 38.1 139.7)
 		)
@@
 	(wire
 		(pts
-			(xy 76.2 160.02) (xy 38.1 160.02)
+			(xy 31.75 160.02) (xy 76.2 160.02)
 		)
 		(stroke
@@
 		(pts
 			(xy 63.5 139.7) (xy 88.9 139.7)
-		)
-		(stroke
-			(width 0)
-			(type default)
-		)
-	)
-	(wire
-		(pts
-			(xy 38.1 156.21) (xy 38.1 160.02)
 		)
 		(stroke
@@
 	)
 	(symbol
+		(lib_id "SynthStuff:MountingHole_Jack6.35mm_v2")
+		(at 38.1 152.4 0)
+		(unit 1)
+		(exclude_from_sim no)
+		(in_bom no)
+		(on_board yes)
+		(dnp no)
+		(fields_autoplaced yes)
+		(property "Reference" "H18"
+			(at 40.64 149.8599 0)
+			(effects
+				(font
+					(size 1.27 1.27)
+				)
+				(justify left)
+			)
+		)
+		(property "Value" "Mod"
+			(at 40.64 152.4 0)
+			(effects
+				(font
+					(size 1.27 1.27)
+					(thickness 0.254)
+					(bold yes)
+					(italic yes)
+				)
+				(justify left)
+			)
+		)
+		(property "Footprint" "SynthStuff:Jack_6.35mm_Cutout_v3"
+			(at 38.1 152.4 0)
+			(effects
+				(font
+					(size 1.27 1.27)
+				)
+				(hide yes)
+			)
+		)
+		(property "Datasheet" "~"
+			(at 38.1 152.4 0)
+			(effects
+				(font
+					(size 1.27 1.27)
+				)
+				(hide yes)
+			)
+		)
+		(property "Description" "Jack 6.35mm"
+			(at 40.64 154.9399 0)
+			(effects
+				(font
+					(size 1.27 1.27)
+				)
+				(justify left)
+			)
+		)
+		(pin "1"
+		)
+		(instances
+			(project "DMH_Slew_Mk2_PANEL"
+				(path "/a552705f-a9fe-462e-9913-5cfcc08b233c"
+					(reference "H18")
+					(unit 1)
+				)
+			)
+		)
+	)
+	(symbol
 		(lib_id "SynthStuff:MountingHole_ToggleSwitch")
 		(at 88.9 127 0)
@@
 	)
 	(symbol
-		(lib_id "SynthStuff:MountingHole_ToggleSwitch")
-		(at 38.1 152.4 0)
-		(unit 1)
-		(exclude_from_sim no)
-		(in_bom no)
-		(on_board yes)
-		(dnp no)
-		(fields_autoplaced yes)
-		(property "Reference" "H23"
-			(at 40.64 149.8599 0)
-			(effects
-				(font
-					(size 1.27 1.27)
-				)
-				(justify left)
-			)
-		)
-		(property "Value" "R/RF/F"
-			(at 40.64 152.4 0)
-			(effects
-				(font
-					(size 1.27 1.27)
-					(thickness 0.254)
-					(bold yes)
-					(italic yes)
-				)
-				(justify left)
-			)
-		)
-		(property "Footprint" "SynthStuff:Toggle_Switch_TE_Cutout"
-			(at 38.1 152.4 0)
-			(effects
-				(font
-					(size 1.27 1.27)
-				)
-				(hide yes)
-			)
-		)
-		(property "Datasheet" "~"
-			(at 38.1 152.4 0)
-			(effects
-				(font
-					(size 1.27 1.27)
-				)
-				(hide yes)
-			)
-		)
-		(property "Description" "Toggle Switch Mounting Hole"
-			(at 40.64 154.9399 0)
-			(effects
-				(font
-					(size 1.27 1.27)
-				)
-				(justify left)
-			)
-		)
-		(pin "1"
-		)
-		(instances
-			(project "DMH_Slew_PANEL"
-				(path "/a552705f-a9fe-462e-9913-5cfcc08b233c"
-					(reference "H23")
-					(unit 1)
-				)
-			)
-		)
-	)
-	(symbol
 		(lib_id "SynthStuff:MountingHole_Jack6.35mm_Output_v2")
 		(at 63.5 177.8 0)
@@
 			)
 		)
-		(property "Value" "Rise A"
+		(property "Value" "Slew A"
 			(at 40.64 114.3 0)
 			(effects
@@
 			)
 		)
-		(property "Footprint" "SynthStuff:Pot_Cutout_Small"
+		(property "Footprint" "SynthStuff:Pot_Cutout_Medium"
 			(at 38.1 115.57 0)
 			(effects
@@
 					(unit 1)
 				)
-			)
-		)
-	)
-	(symbol
-		(lib_id "SynthStuff:MountingHole_Pot")
-		(at 63.5 115.57 0)
-		(unit 1)
-		(exclude_from_sim no)
-		(in_bom yes)
-		(on_board yes)
-		(dnp no)
-		(fields_autoplaced yes)
-		(property "Reference" "H18"
-			(at 66.04 111.7599 0)
-			(effects
-				(font
-					(size 1.27 1.27)
-				)
-				(justify left)
-			)
-		)
-		(property "Value" "Fall A"
-			(at 66.04 114.3 0)
-			(effects
-				(font
-					(size 1.27 1.27)
-					(thickness 0.254)
-					(bold yes)
-					(italic yes)
-				)
-				(justify left)
-			)
-		)
-		(property "Footprint" "SynthStuff:Pot_Cutout_Small"
-			(at 63.5 115.57 0)
-			(effects
-				(font
-					(size 1.27 1.27)
-				)
-				(hide yes)
-			)
-		)
-		(property "Datasheet" "~"
-			(at 63.5 115.57 0)
-			(effects
-				(font
-					(size 1.27 1.27)
-				)
-				(hide yes)
-			)
-		)
-		(property "Description" "Pot Mounting Hole"
-			(at 66.04 116.8399 0)
-			(effects
-				(font
-					(size 1.27 1.27)
-				)
-				(justify left)
-			)
-		)
-		(pin "1"
-		)
-		(instances
-			(project ""
-				(path "/a552705f-a9fe-462e-9913-5cfcc08b233c"
-					(reference "H18")
-					(unit 1)
-				)
