File: DMH_Slew_Mk2_PCB_Controls/Core_Circuit_B.kicad_sch (KiCad schematic)
At the start: 59 parts, among them J1 TS_Jack_6.35mm_Sw, J11 Conn_02x03_Top_Bottom, J12 Conn_02x06_Top_Bottom, J13 Conn_02x03_Top_Bottom, J14 Conn_02x03_Top_Bottom, J15 Conn_02x06_Top_Bottom, J16 Conn_02x03_Top_Bottom, J17 Conn_01x08, J18 Conn_01x08, J19 Conn_01x08, J2 TS_Jack_6.35mm_Sw, J20 Conn_01x08, J3 TS_Jack_6.35mm_Sw, Q1 BC548, Q2 BC548, Q3 BC558, Q4 BC558, SW1 SW_DPDT_3way, SW2 SW_DPDT, SW3 SPDT_OnOffOn, U1 TL074, U2 TL074

Commit message: Designed Controls PCB
... and removed Mod feature
Parts:
- removed C10, C11, C3, C4: 100nF, Capacitor_THT:C_Disc_D4.3mm_W1.9mm_P5.00mm, symbol Device:C
- removed C14: 22nF, Capacitor_THT:C_Disc_D4.3mm_W1.9mm_P5.00mm, symbol Device:C
- removed C15: 220nF, Capacitor_THT:C_Disc_D4.3mm_W1.9mm_P5.00mm, symbol Device:C
- removed C6, C7, C8: 10pF, Capacitor_THT:C_Disc_D3.0mm_W2.0mm_P2.50mm, symbol Device:C
- removed C9: 2.2nF, Capacitor_THT:C_Disc_D4.3mm_W1.9mm_P5.00mm, symbol Device:C
- removed J1, J2, J3: TS_Jack_6.35mm_Sw, SynthStuff:CUI_MJ-63052A, symbol SynthStuff:TS_Jack_6.35mm_Sw
- removed J11, J13: Conn_02x03_Top_Bottom, Connector_PinHeader_2.54mm:PinHeader_2x03_P2.54mm_Horizontal, symbol Connector_Generic:Conn_02x03_Top_Bottom
- removed J12: Conn_02x06_Top_Bottom, Connector_PinHeader_2.54mm:PinHeader_2x06_P2.54mm_Horizontal, symbol Connector_Generic:Conn_02x06_Top_Bottom
- removed J14, J16: Conn_02x03_Top_Bottom, Connector_PinSocket_2.54mm:PinSocket_2x03_P2.54mm_Vertical, symbol Connector_Generic:Conn_02x03_Top_Bottom
- removed J15: Conn_02x06_Top_Bottom, Connector_PinSocket_2.54mm:PinSocket_2x06_P2.54mm_Vertical, symbol Connector_Generic:Conn_02x06_Top_Bottom
- removed J17, J18, J19, J20: Conn_01x08, Connector_PinHeader_2.54mm:PinHeader_1x08_P2.54mm_Vertical, symbol Connector_Generic:Conn_01x08
- removed Q1, Q2: BC548, Package_TO_SOT_THT:TO-92_Inline, symbol Transistor_BJT:BC548
- removed Q3, Q4: BC558, Package_TO_SOT_THT:TO-92_Inline, symbol Transistor_BJT:BC558
- removed R1, R14, R26: 1k, Resistor_THT:R_Axial_DIN0207_L6.3mm_D2.5mm_P7.62mm_Horizontal, symbol Device:R_US
- removed R10, R11, R12, R13, R16, R2, R22, R23, R5, R6, R7, R8, R9: 100k, Resistor_THT:R_Axial_DIN0207_L6.3mm_D2.5mm_P7.62mm_Horizontal, symbol Device:R_US
- removed R15: 82k, Resistor_THT:R_Axial_DIN0207_L6.3mm_D2.5mm_P7.62mm_Horizontal, symbol Device:R_US
- removed R17: 10k, Resistor_THT:R_Axial_DIN0207_L6.3mm_D2.5mm_P7.62mm_Horizontal, symbol Device:R_US
- removed R18, R19, R20, R21: 1k8, Resistor_THT:R_Axial_DIN0207_L6.3mm_D2.5mm_P7.62mm_Horizontal, symbol Device:R_US
- removed R24, R25: 220k, Resistor_THT:R_Axial_DIN0207_L6.3mm_D2.5mm_P7.62mm_Horizontal, symbol Device:R_US
- removed R3, R4: 56k, Resistor_THT:R_Axial_DIN0207_L6.3mm_D2.5mm_P7.62mm_Horizontal, symbol Device:R_US
- removed RV1: 100k, Potentiometer_THT:Potentiometer_Alpha_RD902F-40-00D_Dual_Vertical, symbol Device:R_Potentiometer_Dual_Separate
- removed SW1: SW_DPDT_3way, SynthStuff:Toggle_Switch_2_Poles_TE, symbol SynthStuff:Switch_DPDT
- removed SW2: SW_DPDT, SynthStuff:Toggle_Switch_2_Poles_TE, symbol SynthStuff:Switch_DPDT
- removed SW3: SPDT_OnOffOn, SynthStuff:Toggle_Switch_TE, symbol SynthStuff:SW_SPDT_OnOffOn
- removed U1, U2: TL074, Package_DIP:DIP-14_W7.62mm_Socket, symbol Amplifier_Operational:TL074
- added C17, C21, C22: 10pF, Capacitor_THT:C_Disc_D3.0mm_W2.0mm_P2.50mm, symbol Device:C
- added C18: 220nF, Capacitor_THT:C_Disc_D4.3mm_W1.9mm_P5.00mm, symbol Device:C
- added C19: 22nF, Capacitor_THT:C_Disc_D4.3mm_W1.9mm_P5.00mm, symbol Device:C
- added C20: 2.2nF, Capacitor_THT:C_Disc_D4.3mm_W1.9mm_P5.00mm, symbol Device:C
- added C23, C24, C25, C26: 100nF, Capacitor_THT:C_Disc_D4.3mm_W1.9mm_P5.00mm, symbol Device:C
- added J21, J23, J24, J26: Conn_02x03_Top_Bottom, Connector_PinHeader_2.54mm:PinHeader_2x03_P2.54mm_Horizontal, symbol Connector_Generic:Conn_02x03_Top_Bottom
- added J22, J25: Conn_02x06_Top_Bottom, Connector_PinHeader_2.54mm:PinHeader_2x06_P2.54mm_Horizontal, symbol Connector_Generic:Conn_02x06_Top_Bottom
- added J27, J28: Conn_01x08, Connector_PinHeader_2.54mm:PinHeader_1x08_P2.54mm_Vertical, symbol Connector_Generic:Conn_01x08
- added J29, J30: Conn_01x08, Connector_PinSocket_2.54mm:PinSocket_1x08_P2.54mm_Vertical, symbol Connector_Generic:Conn_01x08
- added J6, J7, J8: TS_Jack_6.35mm_Sw, SynthStuff:CUI_MJ-63052A, symbol SynthStuff:TS_Jack_6.35mm_Sw
- added Q10, Q9: BC558, Package_TO_SOT_THT:TO-92_Inline, symbol Transistor_BJT:BC558
- added Q7, Q8: BC548, Package_TO_SOT_THT:TO-92_Inline, symbol Transistor_BJT:BC548
- added R41, R53: 56k, Resistor_THT:R_Axial_DIN0207_L6.3mm_D2.5mm_P7.62mm_Horizontal, symbol Device:R_US
- added R42, R43, R44, R46, R48, R50, R51, R52, R54, R56, R57, R63, R64: 100k, Resistor_THT:R_Axial_DIN0207_L6.3mm_D2.5mm_P7.62mm_Horizontal, symbol Device:R_US
- added R47, R61, R62: 1k, Resistor_THT:R_Axial_DIN0207_L6.3mm_D2.5mm_P7.62mm_Horizontal, symbol Device:R_US
- added R55, R58: 220k, Resistor_THT:R_Axial_DIN0207_L6.3mm_D2.5mm_P7.62mm_Horizontal, symbol Device:R_US
- added R59, R60, R67, R68: 1k8, Resistor_THT:R_Axial_DIN0207_L6.3mm_D2.5mm_P7.62mm_Horizontal, symbol Device:R_US
- added R65: 82k, Resistor_THT:R_Axial_DIN0207_L6.3mm_D2.5mm_P7.62mm_Horizontal, symbol Device:R_US
- added R66: 10k, Resistor_THT:R_Axial_DIN0207_L6.3mm_D2.5mm_P7.62mm_Horizontal, symbol Device:R_US
- added RV3, RV4: 100k, SynthStuff:Potentiometer_Alpha_RD901F-40-00D_Single_Vertical, symbol Device:R_Potentiometer_US
- added SW4: SW_DPDT_3way, SynthStuff:Toggle_Switch_2_Poles_TE, symbol SynthStuff:Switch_DPDT
- added SW5: SW_DPDT, SynthStuff:Toggle_Switch_2_Poles_TE, symbol SynthStuff:Switch_DPDT
- added SW6: SPDT_OnOffOn, SynthStuff:Toggle_Switch_TE, symbol SynthStuff:SW_SPDT_OnOffOn
- added U3, U4: TL074, Package_DIP:DIP-14_W7.62mm_Socket, symbol Amplifier_Operational:TL074
Connections:
- net +10V: now also J21.2 (Pin_2), J24.2 (Pin_2), J27.5 (Pin_5), J29.5 (Pin_5), J7.TN, R55.1, R58.1, SW4.1 (A), SW4.6 (C), SW5.4 (A)
- net +12V: now also C23.1, C25.1, J21.1 (Pin_1), J24.1 (Pin_1), U3.4 (V+), U4.4 (V+)
- net -12V: now also C24.2, C26.2, J21.3 (Pin_3), J21.4 (Pin_4), J24.3 (Pin_3), J24.4 (Pin_4), U3.11 (V-), U4.11 (V-)
- net GND: now also C23.2, C24.1, C25.2, C26.1, J21.5 (Pin_5), J21.6 (Pin_6), J22.5 (Pin_5), J22.6 (Pin_6), J24.5 (Pin_5), J24.6 (Pin_6), J25.5 (Pin_5), J25.6 (Pin_6), J27.1 (Pin_1), J27.7 (Pin_7), J27.8 (Pin_8), J28.8 (Pin_8), J29.1 (Pin_1), J29.7 (Pin_7), J29.8 (Pin_8), J30.8 (Pin_8), J6.S, J7.S, J8.S, R51.2, R52.2, R59.1, R60.2, R64.2, R67.1, R68.2, RV3.1, RV4.1, SW5.3 (C), SW5.6 (C), U4.12 (+), U4.5 (+)
- new net: R47.1, R51.1, U3.3 (+)
- new net: C21.1, R62.1, U4.9 (-)
- new net: C21.2, R63.2, R65.1, U4.8
- new net: R53.2, RV4.3, SW4.2 (B)
- new net: C22.1, Q10.1 (C), Q7.1 (C), R63.1, U4.13 (-)
- new net: Q10.2 (B), R68.1
- new net: Q10.3 (E), Q7.3 (E), Q8.3 (E), Q9.3 (E), R66.1
- new net: R41.2, RV3.3, SW4.5 (B)
- new net: C18.1, C19.1, C20.1, Q8.1 (C), Q9.1 (C), U4.6 (-)
- new net: R61.2, U4.7
- new net: R48.1, R52.1, U4.3 (+)
- new net: C17.1, R43.2, R46.1, U4.2 (-)
- new net: C22.2, R66.2, U4.14
- new net B_CV_Buff_C: J29.6 (Pin_6), SW4.3 (C), SW4.4 (A)
- new net B_CV_Buff_M: J25.4 (Pin_4), J27.6 (Pin_6)
- new net B_CV_Buff_S: J22.4 (Pin_4), U3.1, U3.2 (-)
- new net B_CV_In_Jack_M: J26.5 (Pin_5), J7.T
- new net B_CV_In_Jack_S: J23.5 (Pin_5), R47.2
- new net B_Comp_-R: Q8.2 (B), R44.1, R50.1, R67.2
- new net B_Comp_F: Q9.2 (B), R42.1, R57.2, R58.2, R60.1
- new net B_Comp_R: Q7.2 (B), R54.1, R55.2, R56.2, R59.2
- new net B_Diff_Amp_C: J29.2 (Pin_2), SW5.1 (A)
- new net B_Diff_Amp_M: J25.1 (Pin_1), J27.2 (Pin_2)
- new net B_Diff_Amp_S: C17.2, J22.1 (Pin_1), R43.1, U4.1
- new net B_F_Gate_Jack_M: J26.1 (Pin_1)
- new net B_F_Gate_Jack_S: J23.1 (Pin_1)
- new net B_F_LED_C: J30.4 (Pin_4)
- new net B_F_LED_M: J25.10 (Pin_10), J28.4 (Pin_4)
- new net B_F_LED_S: J22.10 (Pin_10)
- new net B_Fall_CV_C: J29.4 (Pin_4), R41.1, RV3.2
- new net B_Fall_CV_M: J25.3 (Pin_3), J27.4 (Pin_4)
- new net B_Fall_CV_S: J22.3 (Pin_3), R57.1
- new net B_In_Jack_TN_M: J6.TN
- new net B_Input_Jack_M: J26.4 (Pin_4), J6.T
- new net B_Input_Jack_S: J23.4 (Pin_4), R48.2, R64.1, U4.10 (+)
- new net B_LinLog_Sw_p2_C: J30.2 (Pin_2), SW5.2 (B)
- new net B_LinLog_Sw_p2_M: J25.8 (Pin_8), J28.2 (Pin_2)
- new net B_LinLog_Sw_p2_S: J22.8 (Pin_8), R42.2, R44.2
- new net B_LinLog_Sw_p5_C: J30.1 (Pin_1), SW5.5 (B)
- new net B_LinLog_Sw_p5_M: J25.7 (Pin_7), J28.1 (Pin_1)
- new net B_LinLog_Sw_p5_S: J22.7 (Pin_7), R50.2, R54.2
- new net B_Loopback_M: J26.3 (Pin_3)
- new net B_Loopback_S: J23.3 (Pin_3), R65.2
- new net B_Out_Jack_C: J30.6 (Pin_6), SW6.2 (B)
- new net B_Out_Jack_M: J26.6 (Pin_6), J28.6 (Pin_6), J8.T
- new net B_Out_Jack_S: C20.2, J23.6 (Pin_6), R46.2, R61.1, R62.2
- new net B_Out_Jack_TN_M: J8.TN
- new net B_R_Gate_Jack_M: J26.2 (Pin_2)
- new net B_R_Gate_Jack_S: J23.2 (Pin_2)
- new net B_R_LED_C: J30.3 (Pin_3)
- new net B_R_LED_M: J25.9 (Pin_9), J28.3 (Pin_3)
- new net B_R_LED_S: J22.9 (Pin_9)
- new net B_Rise_CV_C: J29.3 (Pin_3), R53.1, RV4.2
- new net B_Rise_CV_M: J25.2 (Pin_2), J27.3 (Pin_3)
- new net B_Rise_CV_S: J22.2 (Pin_2), R56.1
- new net B_Rng_Sw_p1_C: J30.7 (Pin_7), SW6.1 (A)
- new net B_Rng_Sw_p1_M: J25.12 (Pin_12), J28.7 (Pin_7)
- new net B_Rng_Sw_p1_S: C19.2, J22.12 (Pin_12)
- new net B_Rng_Sw_p3_C: J30.5 (Pin_5), SW6.3 (C)
- new net B_Rng_Sw_p3_M: J25.11 (Pin_11), J28.5 (Pin_5)
- new net B_Rng_Sw_p3_S: C18.2, J22.11 (Pin_11)
