File: DMH_Slew_Mk2_PCB_Controls/DMH_Slew_Mk2_PCB_Controls.kicad_pcb (KiCad board)
At the start: 2 copper layers, 48 x 141 mm, 21 parts, among them J19 Conn_01x08, J20 Conn_01x08, J29 Conn_01x08, J30 Conn_01x08, SW1 SW_DPDT_3way, SW2 SW_DPDT, SW3 SPDT_OnOffOn, SW4 SW_DPDT_3way, SW5 SW_DPDT, SW6 SPDT_OnOffOn

Commit message: Corrected gate outs and CV dest switch locations in PCBs
Parts:
- moved SW1 33.0 mm to (91.5, 159.2)
- moved SW4 33.0 mm to (91.5, 175.8)
Routing:
- net A_CV_Buff_C: track 128.0 -> 141.5 mm
- net Net-(R41-Pad2): track 67.8 -> 56.8 mm
- net B_CV_Buff_C: track 94.1 -> 98.0 mm
- net Net-(R4-Pad2): track 132.7 -> 130.4 mm
- net Net-(R3-Pad2): track 129.1 -> 131.3 mm
- net Net-(R53-Pad2): track 94.2 -> 96.4 mm
Other:
- board size 48 x 141 mm -> 49 x 141 mm
- board text added: "Mk2.1 - July 2026"
- board text removed: "Mk2.0 - April 2026"
