File: DMH_Slew_Mk2_PCB_Main/DMH_Slew_Mk2_PCB_Main.kicad_pcb (KiCad board)
At the start: 2 copper layers, 48 x 175 mm, 33 parts, among them J0 Conn_01x01, J1 TS_Jack_6.35mm_Sw, J10 TS_Jack_6.35mm_Sw, J100 IDC_02x08, J14 Conn_02x03_Top_Bottom, J15 Conn_02x06_Top_Bottom, J16 Conn_02x03_Top_Bottom, J17 Conn_01x08, J18 Conn_01x08, J2 TS_Jack_6.35mm_Sw, J200 IDC_02x05, J24 Conn_02x03_Top_Bottom, J25 Conn_02x06_Top_Bottom, J26 Conn_02x03_Top_Bottom, J27 Conn_01x08, J28 Conn_01x08, J3 TS_Jack_6.35mm_Sw, J4 TS_Jack_6.35mm_Sw, J5 TS_Jack_6.35mm_Sw, J6 TS_Jack_6.35mm_Sw, J7 TS_Jack_6.35mm_Sw, J8 TS_Jack_6.35mm_Sw, J9 TS_Jack_6.35mm_Sw, U10 LM4040LP-10

Commit message: Designed Controls PCB
... and removed Mod feature
Parts:
- moved J18 26.0 mm to (97.2, 50.0)
Routing:
- net A_LinLog_Sw_p5_M: track 53.6 -> 79.6 mm
- net A_F_LED_M: track 45.5 -> 71.5 mm
- net A_LinLog_Sw_p2_M: track 48.8 -> 74.8 mm
- net A_R_LED_M: track 50.2 -> 76.2 mm
- net A_Rng_Sw_p3_M: track 46.8 -> 72.8 mm
- net A_Rng_Sw_p1_M: track 39.5 -> 65.5 mm
- net A_Out_Jack_M: track 151.3 -> 177.2 mm
- net -12V: track 65.7 -> 64.7 mm
Other:
- board text added: "Mk2.0 - April 2026"
- board text removed: "Mk1.1 - April 2026"
