File: DMH_Slew_Mk2_PCB_Main/Core_Circuit_A.kicad_sch (KiCad schematic)
At the start: 59 parts, among them J1 TS_Jack_6.35mm_Sw, J11 Conn_02x03_Top_Bottom, J12 Conn_02x06_Top_Bottom, J13 Conn_02x03_Top_Bottom, J14 Conn_02x03_Top_Bottom, J15 Conn_02x06_Top_Bottom, J16 Conn_02x03_Top_Bottom, J17 Conn_01x08, J18 Conn_01x08, J19 Conn_01x08, J2 TS_Jack_6.35mm_Sw, J20 Conn_01x08, J3 TS_Jack_6.35mm_Sw, Q1 BC548, Q2 BC548, Q3 BC558, Q4 BC558, SW1 SW_DPDT_3way, SW2 SW_DPDT, SW3 SPDT_OnOffOn, U1 TL074, U2 TL074

Commit message: Corrected gate outs and CV dest switch locations in PCBs
Parts:
- J1, J2, J3: footprint SynthStuff:CUI_MJ-63052A -> SynthStuff:CUI_SJ-63083D; symbol SynthStuff:TS_Jack_6.35mm_Sw -> SynthStuff:TRS_Jack_6.35mm_Sw
Connections:
- no-connect marks 0 -> 6
Changed lines of the file:
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@@
 		(color 0 0 0 0)
 	)
+	(no_connect
+		(at 350.52 119.38)
+	)
+	(no_connect
+		(at 55.88 157.48)
+	)
+	(no_connect
+		(at 350.52 121.92)
+	)
+	(no_connect
+		(at 43.18 77.47)
+	)
+	(no_connect
+		(at 43.18 74.93)
+	)
+	(no_connect
+		(at 55.88 160.02)
+	)
 	(wire
 		(pts
@@
 	(wire
 		(pts
-			(xy 349.25 129.54) (xy 349.25 130.81)
+			(xy 347.98 129.54) (xy 347.98 130.81)
 		)
 		(stroke
@@
 	(wire
 		(pts
-			(xy 43.18 80.01) (xy 44.45 80.01)
+			(xy 43.18 80.01) (xy 45.72 80.01)
 		)
 		(stroke
@@
 	(wire
 		(pts
-			(xy 43.18 85.09) (xy 44.45 85.09)
+			(xy 43.18 85.09) (xy 45.72 85.09)
 		)
 		(stroke
@@
 	(wire
 		(pts
-			(xy 350.52 129.54) (xy 349.25 129.54)
+			(xy 350.52 129.54) (xy 347.98 129.54)
 		)
 		(stroke
@@
 	(wire
 		(pts
-			(xy 44.45 85.09) (xy 44.45 86.36)
+			(xy 45.72 85.09) (xy 45.72 86.36)
 		)
 		(stroke
@@
 	(wire
 		(pts
-			(xy 44.45 80.01) (xy 44.45 76.2)
+			(xy 45.72 80.01) (xy 45.72 72.39)
 		)
 		(stroke
@@
 		(polyline
 			(pts
-				(xy 45.085 152.4) (xy 79.375 152.4) (xy 79.375 198.12) (xy 45.085 198.12)
+				(xy 38.1 152.4) (xy 76.2 152.4) (xy 76.2 203.2) (xy 38.1 203.2)
 			)
 			(stroke
@@
 		(polyline
 			(pts
-				(xy 30.48 64.77) (xy 50.8 64.77) (xy 50.8 95.25) (xy 30.48 95.25)
+				(xy 25.4 63.5) (xy 50.8 63.5) (xy 50.8 101.6) (xy 25.4 101.6)
 			)
 			(stroke
@@
 		(polyline
 			(pts
-				(xy 327.66 114.3) (xy 361.95 114.3) (xy 361.9499 139.7) (xy 327.6599 139.7)
+				(xy 327.66 114.3) (xy 370.84 114.3) (xy 370.8399 139.7) (xy 327.6599 139.7)
 			)
 			(stroke
@@
 		(length 2.54)
 		(shape round)
-		(at 30.48 64.77 0)
+		(at 26.67 63.5 0)
 		(fields_autoplaced yes)
 		(effects
@@
 		)
 		(property "Component Class" "Main PCB"
-			(at 31.1785 62.23 0)
+			(at 27.3685 60.96 0)
 			(show_name no)
 			(do_not_autoplace no)
@@
 	(symbol
 		(lib_id "power:GND")
-		(at 44.45 86.36 0)
+		(at 45.72 86.36 0)
 		(unit 1)
 		(body_style 1)
@@
 		(fields_autoplaced yes)
 		(property "Reference" "#PWR05"
-			(at 44.45 92.71 0)
+			(at 45.72 92.71 0)
 			(hide yes)
 			(show_name no)
@@
 		)
 		(property "Value" "GND"
-			(at 44.45 91.44 0)
+			(at 45.72 91.44 0)
 			(show_name no)
 			(do_not_autoplace no)
@@
 		)
 		(property "Footprint" ""
-			(at 44.45 86.36 0)
+			(at 45.72 86.36 0)
 			(hide yes)
 			(show_name no)
@@
 		)
 		(property "Datasheet" ""
-			(at 44.45 86.36 0)
+			(at 45.72 86.36 0)
 			(hide yes)
 			(show_name no)
@@
 		)
 		(property "Description" "Power symbol creates a global label with name \"GND\" , ground"
-			(at 44.45 86.36 0)
+			(at 45.72 86.36 0)
 			(hide yes)
 			(show_name no)
@@
 	(symbol
 		(lib_id "power:+VDC")
-		(at 44.45 76.2 0)
+		(at 45.72 72.39 0)
 		(unit 1)
 		(body_style 1)
@@
 		(fields_autoplaced yes)
 		(property "Reference" "#PWR03"
-			(at 44.45 78.74 0)
+			(at 45.72 74.93 0)
 			(hide yes)
 			(show_name no)
@@
 		)
 		(property "Value" "+10V"
-			(at 44.45 68.58 0)
+			(at 45.72 64.77 0)
 			(show_name no)
 			(do_not_autoplace no)
@@
 		)
 		(property "Footprint" ""
-			(at 44.45 76.2 0)
+			(at 45.72 72.39 0)
 			(hide yes)
 			(show_name no)
@@
 		)
 		(property "Datasheet" ""
-			(at 44.45 76.2 0)
+			(at 45.72 72.39 0)
 			(hide yes)
 			(show_name no)
@@
 		)
 		(property "Description" "Power symbol creates a global label with name \"+VDC\""
-			(at 44.45 76.2 0)
+			(at 45.72 72.39 0)
 			(hide yes)
 			(show_name no)
@@
 		)
 		(property "Function" ""
-			(at 44.45 76.2 0)
+			(at 45.72 72.39 0)
 			(show_name no)
 			(do_not_autoplace no)
@@
 	(symbol
 		(lib_id "power:GND")
-		(at 349.25 130.81 0)
+		(at 347.98 130.81 0)
 		(unit 1)
 		(body_style 1)
@@
 		(fields_autoplaced yes)
 		(property "Reference" "#PWR029"
-			(at 349.25 137.16 0)
+			(at 347.98 137.16 0)
 			(hide yes)
 			(show_name no)
@@
 		)
 		(property "Value" "GND"
-			(at 349.25 135.89 0)
+			(at 347.98 135.89 0)
 			(show_name no)
 			(do_not_autoplace no)
@@
 		)
 		(property "Footprint" ""
-			(at 349.25 130.81 0)
+			(at 347.98 130.81 0)
 			(hide yes)
 			(show_name no)
@@
 		)
 		(property "Datasheet" ""
-			(at 349.25 130.81 0)
+			(at 347.98 130.81 0)
 			(hide yes)
 			(show_name no)
@@
 		)
 		(property "Description" "Power symbol creates a global label with name \"GND\" , ground"
-			(at 349.25 130.81 0)
+			(at 347.98 130.81 0)
 			(hide yes)
 			(show_name no)
@@
 	)
 	(symbol
-		(lib_id "SynthStuff:TS_Jack_6.35mm_Sw")
-		(at 355.6 127 180)
+		(lib_id "SynthStuff:TRS_Jack_6.35mm_Sw")
+		(at 359.41 124.46 0)
+		(mirror y)
 		(unit 1)
 		(body_style 1)
@@
 		(dnp no)
 		(property "Reference" "J3"
-			(at 355.6 132.588 0)
+			(at 359.41 116.84 0)
 			(show_name no)
 			(do_not_autoplace no)
@@
 		)
 		(property "Value" "TS_Jack_6.35mm_Sw"
-			(at 356.235 133.35 0)
+			(at 367.03 132.842 0)
 			(hide yes)
 			(show_name no)
@@
 					(size 1.27 1.27)
 				)
+				(justify left top)
 			)
 		)
-		(property "Footprint" "SynthStuff:CUI_MJ-63052A"
-			(at 355.6 127 0)
+		(property "Footprint" "SynthStuff:CUI_SJ-63083D"
+			(at 359.41 124.46 0)
 			(hide yes)
 			(show_name no)
@@
 					(size 1.27 1.27)
 				)
+				(justify bottom)
 			)
 		)
 		(property "Datasheet" ""
-			(at 355.6 127 0)
+			(at 359.41 124.46 0)
 			(hide yes)
 			(show_name no)
@@
 		)
 		(property "Description" "Audio Jack, 2 Poles (Mono / TS), Switched T Pole (Normalling), 6.35mm, 1/4inch"
-			(at 355.6 127 0)
+			(at 359.41 124.46 0)
 			(hide yes)
 			(show_name no)
@@
 		)
 		(property "Function" "Output A"
-			(at 355.6 119.888 0)
+			(at 359.41 132.588 0)
 			(show_name no)
 			(do_not_autoplace no)
@@
 		(pin "T"
 		)
+		(pin "R"
+		)
+		(pin "RN"
+		)
 		(instances
 			(project "DMH_Slew_Mk2_PCB_Main"
@@
 	)
 	(symbol
-		(lib_id "SynthStuff:TS_Jack_6.35mm_Sw")
-		(at 38.1 82.55 0)
-		(mirror x)
+		(lib_id "SynthStuff:TRS_Jack_6.35mm_Sw")
+		(at 34.29 80.01 0)
 		(unit 1)
 		(body_style 1)
@@
 		(dnp no)
 		(property "Reference" "J2"
-			(at 38.1 88.138 0)
+			(at 34.29 72.136 0)
 			(show_name no)
 			(do_not_autoplace no)
@@
 		)
 		(property "Value" "TS_Jack_6.35mm_Sw"
-			(at 37.465 88.9 0)
+			(at 26.67 88.392 0)
 			(hide yes)
 			(show_name no)
@@
 					(size 1.27 1.27)
 				)
+				(justify left top)
 			)
 		)
-		(property "Footprint" "SynthStuff:CUI_MJ-63052A"
-			(at 38.1 82.55 0)
+		(property "Footprint" "SynthStuff:CUI_SJ-63083D"
+			(at 34.29 80.01 0)
 			(hide yes)
 			(show_name no)
@@
 					(size 1.27 1.27)
 				)
+				(justify bottom)
 			)
 		)
 		(property "Datasheet" ""
-			(at 38.1 82.55 0)
+			(at 34.29 80.01 0)
 			(hide yes)
 			(show_name no)
@@
 		)
 		(property "Description" "Audio Jack, 2 Poles (Mono / TS), Switched T Pole (Normalling), 6.35mm, 1/4inch"
-			(at 38.1 82.55 0)
+			(at 34.29 80.01 0)
 			(hide yes)
 			(show_name no)
@@
 		)
 		(property "Function" "CV A In"
-			(at 38.1 75.438 0)
+			(at 34.29 88.138 0)
 			(show_name no)
 			(do_not_autoplace no)
@@
 		(pin "T"
 		)
+		(pin "R"
+		)
+		(pin "RN"
+		)
 		(instances
 			(project "DMH_Slew_Mk2_PCB_Main"
@@
 	)
 	(symbol
-		(lib_id "SynthStuff:TS_Jack_6.35mm_Sw")
-		(at 50.8 165.1 0)
-		(mirror x)
+		(lib_id "SynthStuff:TRS_Jack_6.35mm_Sw")
+		(at 46.99 162.56 0)
 		(unit 1)
 		(body_style 1)
@@
 		(dnp no)
 		(property "Reference" "J1"
-			(at 50.8 170.942 0)
+			(at 46.99 154.94 0)
 			(show_name no)
 			(do_not_autoplace no)
@@
 		)
 		(property "Value" "TS_Jack_6.35mm_Sw"
-			(at 50.165 171.45 0)
+			(at 39.37 170.942 0)
 			(hide yes)
 			(show_name no)
@@
 					(size 1.27 1.27)
 				)
+				(justify left top)
 			)
 		)
-		(property "Footprint" "SynthStuff:CUI_MJ-63052A"
-			(at 50.8 165.1 0)
+		(property "Footprint" "SynthStuff:CUI_SJ-63083D"
+			(at 46.99 162.56 0)
 			(hide yes)
 			(show_name no)
@@
 					(size 1.27 1.27)
 				)
+				(justify bottom)
 			)
 		)
 		(property "Datasheet" ""
-			(at 50.8 165.1 0)
+			(at 46.99 162.56 0)
 			(hide yes)
 			(show_name no)
@@
 		)
 		(property "Description" "Audio Jack, 2 Poles (Mono / TS), Switched T Pole (Normalling), 6.35mm, 1/4inch"
-			(at 50.8 165.1 0)
+			(at 46.99 162.56 0)
 			(hide yes)
 			(show_name no)
@@
 		)
 		(property "Function" "Input A"
-			(at 50.8 157.988 0)
+			(at 46.99 170.688 0)
 			(show_name no)
 			(do_not_autoplace no)
@@
 		(pin "T"
 		)
+		(pin "R"
+		)
+		(pin "RN"
+		)
 		(instances
