File: DMH_Slew_Mk2_PCB_Main/Core_Circuit_B.kicad_sch (KiCad schematic)
At the start: 60 parts, among them J21 Conn_02x03_Top_Bottom, J22 Conn_02x06_Top_Bottom, J23 Conn_02x03_Top_Bottom, J24 Conn_02x03_Top_Bottom, J25 Conn_02x06_Top_Bottom, J26 Conn_02x03_Top_Bottom, J27 Conn_01x08, J28 Conn_01x08, J29 Conn_01x08, J30 Conn_01x08, J6 TS_Jack_6.35mm_Sw, J7 TS_Jack_6.35mm_Sw, J8 TS_Jack_6.35mm_Sw, Q10 BC558, Q7 BC548, Q8 BC548, Q9 BC558, SW4 SW_DPDT_3way, SW5 SW_DPDT, SW6 SPDT_OnOffOn, U3 TL074, U4 TL074

Commit message: Corrected gate outs and CV dest switch locations in PCBs
Parts:
- J6, J7, J8: footprint SynthStuff:CUI_MJ-63052A -> SynthStuff:CUI_SJ-63083D; symbol SynthStuff:TS_Jack_6.35mm_Sw -> SynthStuff:TRS_Jack_6.35mm_Sw
Connections:
- no-connect marks 0 -> 6
Changed lines of the file:
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@@
 		(color 0 0 0 0)
 	)
+	(no_connect
+		(at 350.52 121.92)
+	)
+	(no_connect
+		(at 41.91 74.93)
+	)
+	(no_connect
+		(at 41.91 77.47)
+	)
+	(no_connect
+		(at 55.88 157.48)
+	)
+	(no_connect
+		(at 350.52 119.38)
+	)
+	(no_connect
+		(at 55.88 160.02)
+	)
 	(wire
 		(pts
@@
 	(wire
 		(pts
-			(xy 43.18 82.55) (xy 53.34 82.55)
-		)
-		(stroke
-			(width 0)
-			(type default)
-		)
-	)
-	(wire
-		(pts
 			(xy 205.74 139.7) (xy 203.2 139.7)
 		)
@@
 	(wire
 		(pts
+			(xy 41.91 80.01) (xy 45.72 80.01)
+		)
+		(stroke
+			(width 0)
+			(type default)
+		)
+	)
+	(wire
+		(pts
 			(xy 154.94 97.79) (xy 154.94 91.44)
 		)
@@
 	(wire
 		(pts
-			(xy 43.18 85.09) (xy 44.45 85.09)
+			(xy 264.16 88.9) (xy 266.7 88.9)
 		)
 		(stroke
@@
 	(wire
 		(pts
-			(xy 264.16 88.9) (xy 266.7 88.9)
+			(xy 213.36 255.27) (xy 215.9 255.27)
 		)
 		(stroke
@@
 	(wire
 		(pts
-			(xy 213.36 255.27) (xy 215.9 255.27)
+			(xy 45.72 80.01) (xy 45.72 76.2)
 		)
 		(stroke
@@
 	(wire
 		(pts
-			(xy 44.45 80.01) (xy 44.45 76.2)
+			(xy 38.1 231.14) (xy 44.45 231.14)
 		)
 		(stroke
@@
 	(wire
 		(pts
-			(xy 38.1 231.14) (xy 44.45 231.14)
+			(xy 226.06 139.7) (xy 228.6 139.7)
 		)
 		(stroke
@@
 	(wire
 		(pts
-			(xy 226.06 139.7) (xy 228.6 139.7)
+			(xy 41.91 85.09) (xy 45.72 85.09)
 		)
 		(stroke
@@
 	(wire
 		(pts
-			(xy 44.45 85.09) (xy 44.45 86.36)
+			(xy 45.72 85.09) (xy 45.72 86.36)
 		)
 		(stroke
@@
 	(wire
 		(pts
-			(xy 43.18 80.01) (xy 44.45 80.01)
+			(xy 342.9 77.47) (xy 349.25 77.47)
 		)
 		(stroke
@@
 	(wire
 		(pts
-			(xy 342.9 77.47) (xy 349.25 77.47)
+			(xy 264.16 135.89) (xy 266.7 135.89)
 		)
 		(stroke
@@
 	(wire
 		(pts
-			(xy 264.16 135.89) (xy 266.7 135.89)
+			(xy 41.91 82.55) (xy 53.34 82.55)
 		)
 		(stroke
@@
 		(polyline
 			(pts
-				(xy 327.66 114.3) (xy 361.95 114.3) (xy 361.95 139.7) (xy 327.66 139.7)
+				(xy 327.66 114.3) (xy 370.84 114.3) (xy 370.84 139.7) (xy 327.66 139.7)
 			)
 			(stroke
@@
 		(polyline
 			(pts
-				(xy 44.45 152.4) (xy 80.01 152.4) (xy 80.01 198.12) (xy 44.45 198.12)
+				(xy 36.83 152.4) (xy 80.01 152.4) (xy 80.01 198.12) (xy 36.83 198.12)
 			)
 			(stroke
@@
 		(polyline
 			(pts
-				(xy 30.48 64.77) (xy 50.8 64.77) (xy 50.8 95.25) (xy 30.48 95.25)
+				(xy 19.05 64.77) (xy 50.8 64.77) (xy 50.8 95.25) (xy 19.05 95.25)
 			)
 			(stroke
@@
 		(length 2.54)
 		(shape round)
-		(at 30.48 64.77 0)
+		(at 21.59 64.77 0)
 		(fields_autoplaced yes)
 		(effects
@@
 		)
 		(property "Component Class" "Main PCB"
-			(at 31.1785 62.23 0)
+			(at 22.2885 62.23 0)
 			(show_name no)
 			(do_not_autoplace no)
@@
 	)
 	(symbol
-		(lib_id "SynthStuff:TS_Jack_6.35mm_Sw")
-		(at 38.1 82.55 0)
-		(mirror x)
+		(lib_id "SynthStuff:TRS_Jack_6.35mm_Sw")
+		(at 33.02 80.01 0)
 		(unit 1)
 		(body_style 1)
@@
 		(dnp no)
 		(property "Reference" "J7"
-			(at 38.1 88.138 0)
+			(at 33.02 72.39 0)
 			(show_name no)
 			(do_not_autoplace no)
@@
 		)
 		(property "Value" "TS_Jack_6.35mm_Sw"
-			(at 37.465 88.9 0)
+			(at 25.4 88.392 0)
 			(hide yes)
 			(show_name no)
@@
 					(size 1.27 1.27)
 				)
+				(justify left top)
 			)
 		)
-		(property "Footprint" "SynthStuff:CUI_MJ-63052A"
-			(at 38.1 82.55 0)
+		(property "Footprint" "SynthStuff:CUI_SJ-63083D"
+			(at 33.02 80.01 0)
 			(hide yes)
 			(show_name no)
@@
 					(size 1.27 1.27)
 				)
+				(justify bottom)
 			)
 		)
 		(property "Datasheet" ""
-			(at 38.1 82.55 0)
+			(at 33.02 80.01 0)
 			(hide yes)
 			(show_name no)
@@
 		)
 		(property "Description" "Audio Jack, 2 Poles (Mono / TS), Switched T Pole (Normalling), 6.35mm, 1/4inch"
-			(at 38.1 82.55 0)
+			(at 33.02 80.01 0)
 			(hide yes)
 			(show_name no)
@@
 		)
 		(property "Function" "CV B In"
-			(at 38.1 75.438 0)
+			(at 33.02 88.138 0)
 			(show_name no)
 			(do_not_autoplace no)
@@
 		(pin "T"
 		)
+		(pin "RN"
+		)
+		(pin "R"
+		)
 		(instances
 			(project "DMH_Slew_Mk2_PCB_Main"
@@
 	)
 	(symbol
-		(lib_id "SynthStuff:TS_Jack_6.35mm_Sw")
-		(at 355.6 127 180)
+		(lib_id "SynthStuff:TRS_Jack_6.35mm_Sw")
+		(at 359.41 124.46 0)
+		(mirror y)
 		(unit 1)
 		(body_style 1)
@@
 		(dnp no)
 		(property "Reference" "J8"
-			(at 355.6 132.588 0)
+			(at 359.41 116.84 0)
 			(show_name no)
 			(do_not_autoplace no)
@@
 		)
 		(property "Value" "TS_Jack_6.35mm_Sw"
-			(at 356.235 133.35 0)
+			(at 367.03 132.842 0)
 			(hide yes)
 			(show_name no)
@@
 					(size 1.27 1.27)
 				)
+				(justify left top)
 			)
 		)
-		(property "Footprint" "SynthStuff:CUI_MJ-63052A"
-			(at 355.6 127 0)
+		(property "Footprint" "SynthStuff:CUI_SJ-63083D"
+			(at 359.41 124.46 0)
 			(hide yes)
 			(show_name no)
@@
 					(size 1.27 1.27)
 				)
+				(justify bottom)
 			)
 		)
 		(property "Datasheet" ""
-			(at 355.6 127 0)
+			(at 359.41 124.46 0)
 			(hide yes)
 			(show_name no)
@@
 		)
 		(property "Description" "Audio Jack, 2 Poles (Mono / TS), Switched T Pole (Normalling), 6.35mm, 1/4inch"
-			(at 355.6 127 0)
+			(at 359.41 124.46 0)
 			(hide yes)
 			(show_name no)
@@
 		)
 		(property "Function" "Output B"
-			(at 355.6 119.888 0)
+			(at 359.41 132.588 0)
 			(show_name no)
 			(do_not_autoplace no)
@@
 		(pin "T"
 		)
+		(pin "R"
+		)
+		(pin "RN"
+		)
 		(instances
 			(project "DMH_Slew_Mk2_PCB_Main"
@@
 	(symbol
 		(lib_id "power:GND")
-		(at 44.45 86.36 0)
+		(at 45.72 86.36 0)
 		(unit 1)
 		(body_style 1)
@@
 		(fields_autoplaced yes)
 		(property "Reference" "#PWR051"
-			(at 44.45 92.71 0)
+			(at 45.72 92.71 0)
 			(hide yes)
 			(show_name no)
@@
 		)
 		(property "Value" "GND"
-			(at 44.45 91.44 0)
+			(at 45.72 91.44 0)
 			(show_name no)
 			(do_not_autoplace no)
@@
 		)
 		(property "Footprint" ""
-			(at 44.45 86.36 0)
+			(at 45.72 86.36 0)
 			(hide yes)
 			(show_name no)
@@
 		)
 		(property "Datasheet" ""
-			(at 44.45 86.36 0)
+			(at 45.72 86.36 0)
 			(hide yes)
 			(show_name no)
@@
 		)
 		(property "Description" "Power symbol creates a global label with name \"GND\" , ground"
-			(at 44.45 86.36 0)
+			(at 45.72 86.36 0)
 			(hide yes)
 			(show_name no)
@@
 	)
 	(symbol
-		(lib_id "SynthStuff:TS_Jack_6.35mm_Sw")
-		(at 50.8 165.1 0)
-		(mirror x)
+		(lib_id "SynthStuff:TRS_Jack_6.35mm_Sw")
+		(at 46.99 162.56 0)
 		(unit 1)
 		(body_style 1)
@@
 		(dnp no)
 		(property "Reference" "J6"
-			(at 50.8 170.942 0)
+			(at 46.99 154.94 0)
 			(show_name no)
 			(do_not_autoplace no)
@@
 		)
 		(property "Value" "TS_Jack_6.35mm_Sw"
-			(at 50.165 171.45 0)
+			(at 39.37 170.942 0)
 			(hide yes)
 			(show_name no)
@@
 					(size 1.27 1.27)
 				)
+				(justify left top)
 			)
 		)
-		(property "Footprint" "SynthStuff:CUI_MJ-63052A"
-			(at 50.8 165.1 0)
+		(property "Footprint" "SynthStuff:CUI_SJ-63083D"
+			(at 46.99 162.56 0)
 			(hide yes)
 			(show_name no)
@@
 					(size 1.27 1.27)
 				)
+				(justify bottom)
 			)
 		)
 		(property "Datasheet" ""
-			(at 50.8 165.1 0)
+			(at 46.99 162.56 0)
 			(hide yes)
 			(show_name no)
@@
 		)
 		(property "Description" "Audio Jack, 2 Poles (Mono / TS), Switched T Pole (Normalling), 6.35mm, 1/4inch"
-			(at 50.8 165.1 0)
+			(at 46.99 162.56 0)
 			(hide yes)
 			(show_name no)
@@
 		)
 		(property "Function" "Input B"
-			(at 50.8 157.988 0)
+			(at 46.99 170.688 0)
 			(show_name no)
 			(do_not_autoplace no)
@@
 		(pin "T"
 		)
+		(pin "RN"
+		)
+		(pin "R"
+		)
 		(instances
 			(project "DMH_Slew_Mk2_PCB_Main"
@@
 	(symbol
 		(lib_id "power:+VDC")
-		(at 44.45 76.2 0)
+		(at 45.72 76.2 0)
 		(unit 1)
 		(body_style 1)
@@
 		(fields_autoplaced yes)
 		(property "Reference" "#PWR016"
-			(at 44.45 78.74 0)
+			(at 45.72 78.74 0)
 			(hide yes)
 			(show_name no)
@@
 		)
 		(property "Value" "+10V"
-			(at 44.45 68.58 0)
+			(at 45.72 68.58 0)
 			(show_name no)
 			(do_not_autoplace no)
@@
 		)
 		(property "Footprint" ""
-			(at 44.45 76.2 0)
+			(at 45.72 76.2 0)
 			(hide yes)
 			(show_name no)
@@
 		)
 		(property "Datasheet" ""
-			(at 44.45 76.2 0)
+			(at 45.72 76.2 0)
 			(hide yes)
 			(show_name no)
@@
 		)
 		(property "Description" "Power symbol creates a global label with name \"+VDC\""
-			(at 44.45 76.2 0)
+			(at 45.72 76.2 0)
 			(hide yes)
 			(show_name no)
@@
 		)
 		(property "Function" ""
-			(at 44.45 76.2 0)
+			(at 45.72 76.2 0)
 			(show_name no)
 			(do_not_autoplace no)
