File: DMH_Slew_Mk2_PCB_Main/State_gate_outputs_A.kicad_sch (KiCad schematic)
At the start: 25 parts, among them J4 TS_Jack_6.35mm_Sw, J5 TS_Jack_6.35mm_Sw, Q5 BC548, Q6 BC548, U1 TL074

Commit message: Corrected gate outs and CV dest switch locations in PCBs
Parts:
- J4, J5: footprint SynthStuff:CUI_MJ-63052A -> SynthStuff:CUI_SJ-63083D; symbol SynthStuff:TS_Jack_6.35mm_Sw -> SynthStuff:TRS_Jack_6.35mm_Sw
Connections:
- no-connect marks 0 -> 4
Changed lines of the file:
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@@
 		(color 0 0 0 0)
+	)
+	(no_connect
+		(at 223.52 116.84)
+	)
+	(no_connect
+		(at 223.52 49.53)
+	)
+	(no_connect
+		(at 223.52 52.07)
+	)
+	(no_connect
+		(at 223.52 119.38)
 	)
 	(wire
@@
 		(polyline
 			(pts
-				(xy 194.31 46.99) (xy 234.95 46.99) (xy 234.95 68.58) (xy 194.31 68.58)
+				(xy 194.945 43.18) (xy 241.935 43.18) (xy 241.935 69.85) (xy 194.945 69.85)
 			)
 			(stroke
@@
 		(polyline
 			(pts
-				(xy 194.31 114.3) (xy 234.95 114.3) (xy 234.95 135.89) (xy 194.31 135.89)
+				(xy 194.945 111.76) (xy 241.935 111.76) (xy 241.935 135.89) (xy 194.945 135.89)
 			)
 			(stroke
@@
 		(length 2.54)
 		(shape round)
-		(at 194.31 114.3 0)
+		(at 195.58 111.76 0)
 		(fields_autoplaced yes)
 		(effects
@@
 		)
 		(property "Component Class" "Main PCB"
-			(at 195.0085 111.76 0)
+			(at 196.2785 109.22 0)
 			(show_name no)
 			(do_not_autoplace no)
@@
 		(length 2.54)
 		(shape round)
-		(at 194.31 46.99 0)
+		(at 195.58 43.18 0)
 		(fields_autoplaced yes)
 		(effects
@@
 		)
 		(property "Component Class" "Main PCB"
-			(at 195.0085 44.45 0)
+			(at 196.2785 40.64 0)
 			(show_name no)
 			(do_not_autoplace no)
@@
 	)
 	(symbol
-		(lib_id "SynthStuff:TS_Jack_6.35mm_Sw")
-		(at 228.6 57.15 180)
+		(lib_id "SynthStuff:TRS_Jack_6.35mm_Sw")
+		(at 232.41 54.61 0)
+		(mirror y)
 		(unit 1)
 		(body_style 1)
@@
 		(dnp no)
 		(property "Reference" "J5"
-			(at 228.6 62.738 0)
+			(at 232.41 46.736 0)
 			(show_name no)
 			(do_not_autoplace no)
@@
 		)
 		(property "Value" "TS_Jack_6.35mm_Sw"
-			(at 229.235 63.5 0)
-			(hide yes)
-			(show_name no)
-			(do_not_autoplace no)
-			(effects
-				(font
-					(size 1.27 1.27)
-				)
-			)
-		)
-		(property "Footprint" "SynthStuff:CUI_MJ-63052A"
-			(at 228.6 57.15 0)
-			(hide yes)
-			(show_name no)
-			(do_not_autoplace no)
-			(effects
-				(font
-					(size 1.27 1.27)
-				)
+			(at 240.03 62.992 0)
+			(hide yes)
+			(show_name no)
+			(do_not_autoplace no)
+			(effects
+				(font
+					(size 1.27 1.27)
+				)
+				(justify left top)
+			)
+		)
+		(property "Footprint" "SynthStuff:CUI_SJ-63083D"
+			(at 232.41 54.61 0)
+			(hide yes)
+			(show_name no)
+			(do_not_autoplace no)
+			(effects
+				(font
+					(size 1.27 1.27)
+				)
+				(justify bottom)
 			)
 		)
 		(property "Datasheet" ""
-			(at 228.6 57.15 0)
+			(at 232.41 54.61 0)
 			(hide yes)
 			(show_name no)
@@
 		)
 		(property "Description" "Audio Jack, 2 Poles (Mono / TS), Switched T Pole (Normalling), 6.35mm, 1/4inch"
-			(at 228.6 57.15 0)
+			(at 232.41 54.61 0)
 			(hide yes)
 			(show_name no)
@@
 		)
 		(property "Function" "Falling A"
-			(at 228.6 50.038 0)
+			(at 232.41 62.738 0)
 			(show_name no)
 			(do_not_autoplace no)
@@
 		)
 		(pin "T"
+		)
+		(pin "R"
+		)
+		(pin "RN"
 		)
 		(instances
@@
 	)
 	(symbol
-		(lib_id "SynthStuff:TS_Jack_6.35mm_Sw")
-		(at 228.6 124.46 180)
+		(lib_id "SynthStuff:TRS_Jack_6.35mm_Sw")
+		(at 232.41 121.92 0)
+		(mirror y)
 		(unit 1)
 		(body_style 1)
@@
 		(dnp no)
 		(property "Reference" "J4"
-			(at 228.6 130.048 0)
+			(at 232.41 114.3 0)
 			(show_name no)
 			(do_not_autoplace no)
@@
 		)
 		(property "Value" "TS_Jack_6.35mm_Sw"
-			(at 229.235 130.81 0)
-			(hide yes)
-			(show_name no)
-			(do_not_autoplace no)
-			(effects
-				(font
-					(size 1.27 1.27)
-				)
-			)
-		)
-		(property "Footprint" "SynthStuff:CUI_MJ-63052A"
-			(at 228.6 124.46 0)
-			(hide yes)
-			(show_name no)
-			(do_not_autoplace no)
-			(effects
-				(font
-					(size 1.27 1.27)
-				)
+			(at 240.03 130.302 0)
+			(hide yes)
+			(show_name no)
+			(do_not_autoplace no)
+			(effects
+				(font
+					(size 1.27 1.27)
+				)
+				(justify left top)
+			)
+		)
+		(property "Footprint" "SynthStuff:CUI_SJ-63083D"
+			(at 232.41 121.92 0)
+			(hide yes)
+			(show_name no)
+			(do_not_autoplace no)
+			(effects
+				(font
+					(size 1.27 1.27)
+				)
+				(justify bottom)
 			)
 		)
 		(property "Datasheet" ""
-			(at 228.6 124.46 0)
+			(at 232.41 121.92 0)
 			(hide yes)
 			(show_name no)
@@
 		)
 		(property "Description" "Audio Jack, 2 Poles (Mono / TS), Switched T Pole (Normalling), 6.35mm, 1/4inch"
-			(at 228.6 124.46 0)
+			(at 232.41 121.92 0)
 			(hide yes)
 			(show_name no)
@@
 		)
 		(property "Function" "Rising A"
-			(at 228.6 117.348 0)
+			(at 232.41 130.048 0)
 			(show_name no)
 			(do_not_autoplace no)
@@
 		(pin "T"
 		)
+		(pin "R"
+		)
+		(pin "RN"
+		)
 		(instances
